File: demos/stickhub/StickHub.kicad_sch (KiCad schematic)
At the start: 94 parts, among them J1 HOST, J2 USB1, J3 USB2, J4 USB3, J5 USB4, J6 USB5, J7 USB6, J8 USB7, J9 EXTGND, U1 MaxLinear_XR22417-48, U2 Dialog_SLG5NT1487V, Y1 12MHz 50ppm 16-20pF

Commit message: 10.0
Other:
- moved on the sheet: C1, C10, C11, C12, C13, C14, C15, C16, C17, C18, C19, C2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
