File: qa/data/pcbnew/length_calculations.kicad_pcb (KiCad board)
At the start: 2 copper layers, 21.8 x 34 mm, 12 parts

Commit message: 10.0
Parts:
- added R13: R, Resistor_SMD:R_0805_2012Metric, F.Cu at (121.4, 80.3)
- added R14: R, Resistor_SMD:R_0805_2012Metric, F.Cu at (136.6, 80.3)
- added R15: R, Resistor_SMD:R_0805_2012Metric, F.Cu at (121.4, 85.2)
- added R16: R, Resistor_SMD:R_0805_2012Metric, B.Cu at (136.6, 85.2)
Routing:
- net Net-(R15-Pad2): track 0.00 -> 13.3 mm, vias 0 -> 3
- net Net-(R13-Pad2): track 0.00 -> 13.3 mm, vias 0 -> 3
Other:
- board size 21.8 x 34 mm -> 21.8 x 43.8 mm
- copper layers 2 -> 4
- board text added: "Single track from pad to pad through internal layer vias. Length 13.3350mm (13.3350mm track, 20.1750mm via)"
- board text added: "Single track from pad to pad through internal layer vias. Length 28.4750mm (13.3350mm track, 15.1400mm via)"
- board text added: "Single track from pad to pad, with pad in via. Length 28.4750mm (13.3350mm track, 15.1400mm via)"
- board text added: "Track from pad to pad with two vias in track. Length 43.6150mm (13.3350mm track, 30.2800mm via)"
- board text added: "Track from pad to pad with via in track. Length 28.4750mm (13.3350mm track, 15.1400mm via)"
- board text removed: "Single track from pad to pad, with pad in via. Length 14.880mm (13.3350mm track, 1.545mm via)"
- board text removed: "Track from pad to pad with two vias in track. Length 16.4250mm (13.3350mm track, 3.0900mm via)"
- board text removed: "Track from pad to pad with via in track. Length 14.880mm (13.3350mm track, 1.545mm via)"
