File: qa/data/pcbnew/time_calculations.kicad_pcb (KiCad board)
At the start: 4 copper layers, 81.9 x 85.1 mm, 16 parts

Commit message: 10.0
Other:
- board text added: "Two layer track + via T = 31.43ps"
- board text removed: "Two layer track + via T = 31.39ps"
Changed lines of the file:
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@@
 (kicad_pcb
-	(version 20250401)
+	(version 20250926)
 	(generator "pcbnew")
 	(generator_version "9.99")
@@
 			(usegerberadvancedattributes yes)
 			(creategerberjobfile yes)
-			(dashed_line_dash_ratio 12.000000)
-			(dashed_line_gap_ratio 3.000000)
+			(dashed_line_dash_ratio 12)
+			(dashed_line_gap_ratio 3)
 			(svgprecision 4)
 			(plotframeref no)
 			(mode 1)
 			(useauxorigin no)
-			(hpglpennumber 1)
-			(hpglpenspeed 20)
-			(hpglpendiameter 15.000000)
 			(pdf_front_fp_property_popups yes)
 			(pdf_back_fp_property_popups yes)
@@
 		)
 	)
-	(gr_text "Two layer track + via\nT = 31.39ps"
+	(gr_text "Two layer track + via\nT = 31.43ps"
 		(at 128.905 71.12 0)
 		(layer "User.1")
